File: Hardware/OSHPark/001.kicad_pcb (KiCad board)
At the start: 2 copper layers, 73.1 x 87.8 mm, 32 parts, among them J1 CONN_01X02, J2 CONN_01X03, J3 CONN_01X03, J4 CONN_02X03, J5 CONN_01X02, U1 LM340MP-5.0/NOPB, U2 ATTINY85-20SU

Commit message: Generated Gerbers Files
Parts:
- moved LED2 0.27 mm to (116.9, 82.9)
Routing:
- net VCC: track 51.9 -> 47.4 mm
Changed lines of the file:
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@@
 (kicad_pcb (version 4) (host pcbnew 4.0.7-e2-6376~58~ubuntu16.04.1)
   (general
-    (links 0)
+    (links 56)
     (no_connects 0)
     (area 77.097479 10.629239 256.622281 146.050001)
     (thickness 1.6)
     (drawings 1017)
-    (tracks 283)
+    (tracks 284)
     (zones 0)
     (modules 32)
@@
     (visible_elements 7FFFFFFF)
     (pcbplotparams
-      (layerselection 0x010f0_ffffffff)
+      (layerselection 0x010f0_80000001)
       (usegerberextensions true)
       (usegerberattributes true)
@@
   )
   (module OSHwi:WS2812B (layer F.Cu)
-    (at 116.9416 83.185)
+    (at 116.8654 82.931)
     (fp_text reference LED2 (at 0.025 0) (layer F.Fab)
       (effects (font (size 1 1) (thickness 0.15)))
@@
   (segment (start 145.505858 103.2256) (end 146.631547 104.351289) (width 0.6096) (layer B.Cu) (net 3))
   (segment (start 146.631547 104.351289) (end 156.36039 104.351289) (width 0.6096) (layer B.Cu) (net 3))
+  (segment (start 134.875 121.92) (end 124.6124 121.92) (width 0.8) (layer B.Cu) (net 4))
+  (segment (start 124.6124 121.92) (end 119.786096 117.093696) (width 0.8) (layer B.Cu) (net 4))
+  (segment (start 119.786096 117.093696) (end 119.786096 110.376167) (width 0.8) (layer B.Cu) (net 4))
+  (segment (start 119.786096 110.376167) (end 119.856535 110.305728) (width 0.8) (layer B.Cu) (net 4))
   (segment (start 122.025 110.5154) (end 121.825 110.5154) (width 0.8) (layer B.Cu) (net 4))
   (segment (start 131.205 101.575) (end 131.205 103.375) (width 0.8) (layer B.Cu) (net 4))
@@
   (segment (start 121.825 110.5154) (end 120.025 110.5154) (width 0.8) (layer B.Cu) (net 4))
   (segment (start 120.025 110.5154) (end 119.7864 110.2768) (width 0.8) (layer B.Cu) (net 4))
-  (segment (start 124.6124 121.92) (end 118.014 115.3216) (width 0.8) (layer B.Cu) (net 4))
-  (segment (start 118.014 115.3216) (end 118.014 106.553) (width 0.8) (layer B.Cu) (net 4))
-  (segment (start 134.875 121.92) (end 124.6124 121.92) (width 0.8) (layer B.Cu) (net 4))
   (segment (start 115.959 106.553) (end 118.014 106.553) (width 0.8) (layer B.Cu) (net 4))
   (segment (start 137.15 124.9272) (end 138.175 123.9022) (width 0.8) (layer B.Cu) (net 5))
