File: Hardware/PCBWay/001.kicad_pcb (KiCad board)
At the start: 2 copper layers, 73.1 x 87.8 mm, 31 parts, among them J1 CONN_01X02, J2 CONN_01X03, J3 CONN_01X03, J4 CONN_02X03, J5 CONN_01X02, U1 LM340MP-5.0/NOPB, U2 ATTINY85-20SU

Commit message: Update Capacitors Value en Voltage Regulator
Parts:
- C1: value 0.22uF -> 4.7uF
- C2: value 0.1uF -> 4.7uF
Changed lines of the file:
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@@
     (links 56)
     (no_connects 0)
-    (area 77.097479 10.629239 256.622281 146.050001)
+    (area 99.401254 53.288629 172.609346 141.218211)
     (thickness 1.6)
     (drawings 1017)
@@
   )
   (layers
-    (0 F.Cu signal)
-    (31 B.Cu signal)
+    (0 F.Cu signal hide)
+    (31 B.Cu signal hide)
     (34 B.Paste user)
     (35 F.Paste user)
-    (36 B.SilkS user)
-    (37 F.SilkS user)
+    (36 B.SilkS user hide)
+    (37 F.SilkS user hide)
     (38 B.Mask user)
     (39 F.Mask user)
@@
       (effects (font (size 1 1) (thickness 0.15)) (justify mirror))
     )
-    (fp_text value 0.22uF (at 0 -2) (layer B.Fab)
+    (fp_text value 4.7uF (at 0 -2) (layer B.Fab)
       (effects (font (size 1 1) (thickness 0.15)) (justify mirror))
     )
@@
       (effects (font (size 1 1) (thickness 0.15)) (justify mirror))
     )
-    (fp_text value 0.1uF (at 0 -2) (layer B.Fab)
-      (effects (font (size 1 1) (thickness 0.15)) (justify mirror))
-    )
+    (fp_text value 4.7uF (at 0 -2) (layer B.Fab)
+      (effects (font (size 1 1) (thickness 0.15)) (justify mirror))
+    )
